Commit message: get transformation to base right. ros industrial usus is root link must be base_link

File: tm_description/urdf/tm1100.urdf.xacro (robot description, xacro)
@@ -276,6 +276,6 @@
     <joint name="${prefix}base-base_link" type="fixed">
       <origin xyz="0 0 0" rpy="0 0 0"/>
-      <parent link="${prefix}base"/>
-      <child link="${prefix}base_link"/>
+      <parent link="${prefix}base_link"/>
+      <child link="${prefix}base"/>
     </joint>
     <!-- Frame coincident with all-zeros TCP on TM controller -->

File: tm_description/urdf/tm1100_robot.urdf.xacro (robot description, xacro)
@@ -12,5 +12,5 @@
   <joint name="world_joint" type="fixed">
     <parent link="world" />
-    <child link="base" />
+    <child link="base_link" />
     <origin xyz="0 0 0" rpy="0 0 0" />
   </joint>

File: tm_description/urdf/tm1100_robot_joint_limited.urdf.xacro (robot description, xacro)
@@ -12,5 +12,5 @@
   <joint name="world_joint" type="fixed">
     <parent link="world" />
-    <child link="base" />
+    <child link="base_link" />
     <origin xyz="0 0 0" rpy="0 0 0" />
   </joint>

File: tm_description/urdf/tm1300.urdf.xacro (robot description, xacro)
@@ -275,6 +275,6 @@
     <joint name="${prefix}base-base_link" type="fixed">
       <origin xyz="0 0 0" rpy="0 0 0"/>
-      <parent link="${prefix}base"/>
-      <child link="${prefix}base_link"/>
+      <parent link="${prefix}base_link"/>
+      <child link="${prefix}base"/>
     </joint>
     <!-- Frame coincident with all-zeros TCP on TM controller -->

File: tm_description/urdf/tm1300_robot.urdf.xacro (robot description, xacro)
@@ -12,5 +12,5 @@
   <joint name="world_joint" type="fixed">
     <parent link="world" />
-    <child link="base" />
+    <child link="base_link" />
     <origin xyz="0 0 0" rpy="0 0 0" />
   </joint>

File: tm_description/urdf/tm1300_robot_joint_limited.urdf.xacro (robot description, xacro)
@@ -12,5 +12,5 @@
   <joint name="world_joint" type="fixed">
     <parent link="world" />
-    <child link="base" />
+    <child link="base_link" />
     <origin xyz="0 0 0" rpy="0 0 0" />
   </joint>

File: tm_description/urdf/tm700.urdf.xacro (robot description, xacro)
@@ -276,6 +276,6 @@
     <joint name="${prefix}base-base_link" type="fixed">
       <origin xyz="0 0 0" rpy="0 0 0"/>
-      <parent link="${prefix}base"/>
-      <child link="${prefix}base_link"/>
+      <parent link="${prefix}base_link"/>
+      <child link="${prefix}base"/>
     </joint>
     <!-- Frame coincident with all-zeros TCP on TM controller -->

File: tm_description/urdf/tm700_robot.urdf.xacro (robot description, xacro)
@@ -12,5 +12,5 @@
   <joint name="world_joint" type="fixed">
     <parent link="world" />
-    <child link="base" />
+    <child link="base_link" />
     <origin xyz="0 0 0" rpy="0 0 0" />
   </joint>

File: tm_description/urdf/tm700_robot_eih.urdf.xacro (robot description, xacro)
@@ -12,5 +12,5 @@
   <joint name="world_joint" type="fixed">
     <parent link="world" />
-    <child link="base" />
+    <child link="base_link" />
     <origin xyz="0 0 0" rpy="0 0 0" />
   </joint>

File: tm_description/urdf/tm700_robot_joint_limited.urdf.xacro (robot description, xacro)
@@ -12,5 +12,5 @@
   <joint name="world_joint" type="fixed">
     <parent link="world" />
-    <child link="base" />
+    <child link="base_link" />
     <origin xyz="0 0 0" rpy="0 0 0" />
   </joint>

File: tm_description/urdf/tm700_robot_joint_limited_eih.urdf.xacro (robot description, xacro)
@@ -12,5 +12,5 @@
   <joint name="world_joint" type="fixed">
     <parent link="world" />
-    <child link="base" />
+    <child link="base_link" />
     <origin xyz="0 0 0" rpy="0 0 0" />
   </joint>

File: tm_description/urdf/tm900.urdf.xacro (robot description, xacro)
@@ -275,6 +275,6 @@
     <joint name="${prefix}base-base_link" type="fixed">
       <origin xyz="0 0 0" rpy="0 0 0"/>
-      <parent link="${prefix}base"/>
-      <child link="${prefix}base_link"/>
+      <parent link="${prefix}base_link"/>
+      <child link="${prefix}base"/>
     </joint>
     <!-- Frame coincident with all-zeros TCP on TM controller -->

File: tm_description/urdf/tm900_robot.urdf.xacro (robot description, xacro)
@@ -12,5 +12,5 @@
   <joint name="world_joint" type="fixed">
     <parent link="world" />
-    <child link="base" />
+    <child link="base_link" />
     <origin xyz="0 0 0" rpy="0 0 0" />
   </joint>

File: tm_description/urdf/tm900_robot_eih.urdf.xacro (robot description, xacro)
@@ -12,5 +12,5 @@
   <joint name="world_joint" type="fixed">
     <parent link="world" />
-    <child link="base" />
+    <child link="base_link" />
     <origin xyz="0 0 0" rpy="0 0 0" />
   </joint>

File: tm_description/urdf/tm900_robot_joint_limited.urdf.xacro (robot description, xacro)
@@ -12,5 +12,5 @@
   <joint name="world_joint" type="fixed">
     <parent link="world" />
-    <child link="base" />
+    <child link="base_link" />
     <origin xyz="0 0 0" rpy="0 0 0" />
   </joint>

File: tm_description/urdf/tm900_robot_joint_limited_eih.urdf.xacro (robot description, xacro)
@@ -12,5 +12,5 @@
   <joint name="world_joint" type="fixed">
     <parent link="world" />
-    <child link="base" />
+    <child link="base_link" />
     <origin xyz="0 0 0" rpy="0 0 0" />
   </joint>
